File: PortBreakoutCapacitive_r3_no_user.brd (EAGLE design)
At the start: 24.4 x 49.8 mm, 10 parts, among them IC1 AT42QT1011-TSHR

Commit message: minor clean-up
Parts:
- C2, C3: value 0.1uF -> 100nF
Changed lines of the file:
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@@
 <attribute name="VALUE" x="6.096" y="17.145" size="0.6096" layer="25" font="vector" align="top-center"/>
 </element>
-<element name="C2" library="rcl" library_urn="urn:adsk.eagle:library:334" package="C1206" package3d_urn="urn:adsk.eagle:package:23618/2" value="0.1uF" x="12.954" y="19.685" smashed="yes" rot="R90">
+<element name="C2" library="rcl" library_urn="urn:adsk.eagle:library:334" package="C1206" package3d_urn="urn:adsk.eagle:package:23618/2" value="100nF" x="12.954" y="19.685" smashed="yes" rot="R90">
 <attribute name="NAME" x="12.954" y="22.225" size="0.6096" layer="25" font="vector" align="bottom-center"/>
 <attribute name="POPULARITY" value="54" x="13.335" y="19.685" size="1.778" layer="27" rot="R90" display="off"/>
@@
 <attribute name="VALUE" x="12.954" y="17.145" size="0.6096" layer="25" font="vector" align="top-center"/>
 </element>
-<element name="C3" library="rcl" library_urn="urn:adsk.eagle:library:334" package="C1206" package3d_urn="urn:adsk.eagle:package:23618/2" value="0.1uF" x="9.525" y="25.781" smashed="yes" rot="R180">
+<element name="C3" library="rcl" library_urn="urn:adsk.eagle:library:334" package="C1206" package3d_urn="urn:adsk.eagle:package:23618/2" value="100nF" x="9.525" y="25.781" smashed="yes" rot="R180">
 <attribute name="NAME" x="9.525" y="26.797" size="0.6096" layer="25" font="vector" align="bottom-center"/>
 <attribute name="POPULARITY" value="54" x="9.525" y="25.781" size="1.778" layer="27" rot="R180" display="off"/>
