File: PortBreakoutCapacitive_r3.brd (EAGLE design)
At the start: 24.4 x 49.8 mm, 10 parts, among them IC1 AT42QT1011-TSHR

Commit message: Revert "rev 4: C1 with lower capacitance"
This reverts commit f0b3ebc7fd996792bcba9bfe078b693bdcbdf926.
Parts:
- C1: value 6.8nF -> 10nF
Other:
- board text added: "rev 3"
- board text removed: "rev 4"
Changed lines of the file:
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@@
 <plain>
 <text x="13.462" y="2.54" size="1.016" layer="21" font="vector" align="top-center">port interface</text>
-<text x="13.335" y="45.466" size="1.27" layer="21" font="vector" rot="R180" align="bottom-center">rev 4</text>
+<text x="13.335" y="45.466" size="1.27" layer="21" font="vector" rot="R180" align="bottom-center">rev 3</text>
 <text x="4.826" y="8.255" size="1.016" layer="21" font="vector" align="top-center">SNS</text>
 <wire x1="1.143" y1="0.762" x2="25.527" y2="0.762" width="0" layer="20"/>
@@
 <attribute name="VALUE" x="3.302" y="17.145" size="0.6096" layer="25" font="vector" align="top-center"/>
 </element>
-<element name="C1" library="rcl" library_urn="urn:adsk.eagle:library:334" package="C1206" package3d_urn="urn:adsk.eagle:package:23618/2" value="6.8nF" x="6.096" y="19.685" smashed="yes" rot="R90">
+<element name="C1" library="rcl" library_urn="urn:adsk.eagle:library:334" package="C1206" package3d_urn="urn:adsk.eagle:package:23618/2" value="10nF" x="6.096" y="19.685" smashed="yes" rot="R90">
 <attribute name="NAME" x="6.096" y="22.225" size="0.6096" layer="25" font="vector" align="bottom-center"/>
 <attribute name="POPULARITY" value="54" x="7.366" y="20.447" size="1.778" layer="27" rot="R90" display="off"/>
